File: storyboard/storyboard.kicad_sch (KiCad schematic)
At the start: 168 parts, among them J1 Debug Breakout, J2 JST-SH 4 Pin, J3 MICROMOD-2222-C, J4 Conn_02x20_Odd_Even, SW1 Switch_1u, SW10 Switch_1u, SW11 Switch_1u, SW12 Switch_1u, SW13 Switch_1u, SW14 Switch_1u, SW15 Switch_1u, SW16 Switch_1u, SW17 Switch_1u, SW18 Switch_1u, SW19 Switch_1u, SW2 Switch_1u, SW20 Switch_1u, SW21 Switch_1u, SW22 Switch_1u, SW23 Switch_1u, SW24 Switch_1u, SW25 Switch_1u, SW26 Switch_1u, SW27 Switch_1u, SW28 Switch_1u, SW29 Switch_1u, SW3 Switch_1u, SW30 Switch_1u, SW31 Switch_1u, SW32 Switch_1u, SW33 Switch_1u, SW34 Switch_1u, SW35 Switch_1u, SW36 Switch_1u, SW37 Switch_1u, SW38 Switch_1u, SW39 Switch_1u, SW4 Switch_1u, SW40 Switch_1u, SW41 Switch_1u, SW42 Switch_1u, SW43 Switch_1u, SW44 Switch_1u, SW45 Switch_1u, SW46 Switch_1u, SW47 Switch_1u, SW48 Switch_1u, SW49 Switch_1u, SW5 Switch_1u, SW50 Switch_1u, SW51 Switch_1u, SW52 Switch_1u, SW53 Switch_1u, SW54 Switch_1u, SW55 Switch_1u, SW56 Switch_1u, SW57 Switch_1u, SW58 Switch_1u, SW59 Switch_1u, SW6 Switch_1u, SW60 Switch_1u, SW61 RESET, SW62 BOOT, SW7 Switch_1u, SW8 Switch_1u, SW9 Switch_1u, U1 74HC164 (SIPO), U2 74HC165 (PISO), U3 74HC165 (PISO), U4 AP7361C-33E

Commit message: add 3d step files for remaining foot prints
Parts:
- added J5: M2.5 Standoff, storyboard:Micromod-Standoff, symbol Connector:Conn_01x01_Female
- J2: value JST-SH 4 Pin -> Pico-EZmate; footprint Connector_JST:JST_SH_SM04B-SRSS-TB_1x04-1MP_P1.00mm_Horizontal -> storyboard:Pico-EZmate 4-pin
- SW61, SW62: footprint Button_Switch_SMD:SW_SPST_TL3305A -> Button_Switch_THT:SW_PUSH_6mm
Connections:
- net GND: now also J5.1 (Pin_1)
Changed lines of the file:
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@@
     (stroke (width 0) (type default) (color 0 0 0 0))
   )
+  (wire (pts (xy 367.03 224.79) (xy 367.03 227.33))
+    (stroke (width 0) (type default) (color 0 0 0 0))
+  )
   (wire (pts (xy 166.37 247.65) (xy 166.37 257.81))
     (stroke (width 0) (type default) (color 0 0 0 0))
@@
     (property "Reference" "SW61" (id 0) (at 256.54 138.43 0))
     (property "Value" "RESET" (id 1) (at 256.54 140.97 0))
-    (property "Footprint" "Button_Switch_SMD:SW_SPST_TL3305A" (id 2) (at 256.54 140.97 0)
+    (property "Footprint" "Button_Switch_THT:SW_PUSH_6mm" (id 2) (at 256.54 140.97 0)
       (effects (font (size 1.27 1.27)) hide)
     )
-    (property "Datasheet" "https://www.digikey.com/en/products/detail/e-switch/TL3305BF260QG/5816185" (id 3) (at 256.54 140.97 0)
+    (property "Datasheet" "https://www.digikey.com/en/products/detail/cui-devices/TS02-66-60-BK-100-SCR-D/15634358?utm_adgroup=&utm_term=&utm_content=" (id 3) (at 256.54 140.97 0)
       (effects (font (size 1.27 1.27)) hide)
     )
@@
     (property "Reference" "SW62" (id 0) (at 264.16 149.86 0))
     (property "Value" "BOOT" (id 1) (at 264.16 152.4 0))
-    (property "Footprint" "Button_Switch_SMD:SW_SPST_TL3305A" (id 2) (at 264.16 152.4 0)
+    (property "Footprint" "Button_Switch_THT:SW_PUSH_6mm" (id 2) (at 264.16 152.4 0)
       (effects (font (size 1.27 1.27)) hide)
     )
-    (property "Datasheet" "https://www.digikey.com/en/products/detail/e-switch/TL3305BF260QG/5816185" (id 3) (at 264.16 152.4 0)
+    (property "Datasheet" "https://www.digikey.com/en/products/detail/cui-devices/TS02-66-60-BK-100-SCR-D/15634358?utm_adgroup=&utm_term=&utm_content=" (id 3) (at 264.16 152.4 0)
       (effects (font (size 1.27 1.27)) hide)
     )
@@
       (effects (font (size 1.27 1.27)) (justify left))
     )
-    (property "Value" "JST-SH 4 Pin" (id 1) (at 309.88 54.6099 0)
+    (property "Value" "Pico-EZmate" (id 1) (at 309.88 54.6099 0)
       (effects (font (size 1.27 1.27)) (justify left))
     )
-    (property "Footprint" "Connector_JST:JST_SH_SM04B-SRSS-TB_1x04-1MP_P1.00mm_Horizontal" (id 2) (at 307.34 52.07 0)
+    (property "Footprint" "storyboard:Pico-EZmate 4-pin" (id 2) (at 307.34 52.07 0)
       (effects (font (size 1.27 1.27)) hide)
     )
-    (property "Datasheet" "~" (id 3) (at 307.34 52.07 0)
+    (property "Datasheet" "https://www.digikey.com/en/products/detail/molex/0781710004/2424925" (id 3) (at 307.34 52.07 0)
       (effects (font (size 1.27 1.27)) hide)
     )
@@
     (pin "2")
   )
+  (symbol (lib_id "power:GND") (at 367.03 227.33 0) (unit 1)
+    (in_bom yes) (on_board yes) (fields_autoplaced)
+    (property "Reference" "#PWR0101" (id 0) (at 367.03 233.68 0)
+      (effects (font (size 1.27 1.27)) hide)
+    )
+    (property "Value" "GND" (id 1) (at 367.03 232.41 0))
+    (property "Footprint" "" (id 2) (at 367.03 227.33 0)
+      (effects (font (size 1.27 1.27)) hide)
+    )
+    (property "Datasheet" "" (id 3) (at 367.03 227.33 0)
+      (effects (font (size 1.27 1.27)) hide)
+    )
+    (pin "1")
+  )
   (symbol (lib_id "power:+3.3V") (at 265.43 48.26 0) (unit 1)
     (in_bom yes) (on_board yes) (fields_autoplaced)
@@
     (pin "2")
   )
+  (symbol (lib_id "Connector:Conn_01x01_Female") (at 372.11 224.79 0) (unit 1)
+    (in_bom yes) (on_board yes) (fields_autoplaced)
+    (property "Reference" "J5" (id 0) (at 373.38 223.5199 0)
+      (effects (font (size 1.27 1.27)) (justify left))
+    )
+    (property "Value" "M2.5 Standoff" (id 1) (at 373.38 226.0599 0)
+      (effects (font (size 1.27 1.27)) (justify left))
+    )
+    (property "Footprint" "storyboard:Micromod-Standoff" (id 2) (at 372.11 224.79 0)
+      (effects (font (size 1.27 1.27)) hide)
+    )
+    (property "Datasheet" "https://www.digikey.com/en/products/detail/w%C3%BCrth-elektronik/9774040151R/5320694?utm_adgroup=General&utm_term=" (id 3) (at 372.11 224.79 0)
+      (effects (font (size 1.27 1.27)) hide)
+    )
+    (pin "1")
+  )
   (symbol (lib_id "Switch:SW_Push") (at 156.21 222.25 0) (unit 1)
     (in_bom yes) (on_board yes) (fields_autoplaced)
@@
       (effects (font (size 0.508 0.508)) hide)
     )
-    (property "Datasheet" "" (id 3) (at 313.69 194.31 0)
+    (property "Datasheet" "https://www.digikey.com/en/products/detail/amphenol-cs-fci/MDT420E03001/5810340" (id 3) (at 313.69 194.31 0)
       (effects (font (size 1.27 1.27)) hide)
     )
@@
       (reference "#PWR047") (unit 1) (value "GND") (footprint "")
     )
+    (path "/25733bf5-cad8-4cf0-b8de-d8be4c3de43f"
+      (reference "#PWR0101") (unit 1) (value "GND") (footprint "")
+    )
     (path "/39f2509c-f884-412c-ba18-e5f920406fac"
       (reference "C1") (unit 1) (value "0.1uF") (footprint "Capacitor_SMD:C_0805_2012Metric")
@@
     )
     (path "/2415dc3c-d1ee-4557-8893-b4607fc8c658"
-      (reference "J2") (unit 1) (value "JST-SH 4 Pin") (footprint "Connector_JST:JST_SH_SM04B-SRSS-TB_1x04-1MP_P1.00mm_Horizontal")
+      (reference "J2") (unit 1) (value "Pico-EZmate") (footprint "storyboard:Pico-EZmate 4-pin")
     )
     (path "/dea6934b-3b47-4910-a45b-119063d57e6c"
@@
       (reference "J4") (unit 1) (value "Conn_02x20_Odd_Even") (footprint "storyboard:Waveshare_ePaper_HAT_352")
     )
+    (path "/b281d559-94ce-4b05-b97d-b3615b82ef39"
+      (reference "J5") (unit 1) (value "M2.5 Standoff") (footprint "storyboard:Micromod-Standoff")
+    )
     (path "/0fe0bc2a-0419-4260-a05a-d39f80967f59"
       (reference "R1") (unit 1) (value "10k") (footprint "Resistor_SMD:R_0805_2012Metric")
@@
     )
     (path "/065a19be-f41e-469c-97bf-cb8cd0ea2c5c"
-      (reference "SW61") (unit 1) (value "RESET") (footprint "Button_Switch_SMD:SW_SPST_TL3305A")
+      (reference "SW61") (unit 1) (value "RESET") (footprint "Button_Switch_THT:SW_PUSH_6mm")
     )
     (path "/20fab8c2-43b9-464e-abc2-f3cfde70931f"
-      (reference "SW62") (unit 1) (value "BOOT") (footprint "Button_Switch_SMD:SW_SPST_TL3305A")
+      (reference "SW62") (unit 1) (value "BOOT") (footprint "Button_Switch_THT:SW_PUSH_6mm")
     )
     (path "/2d5c51a1-3a67-4a18-834e-5ae1905f1acb"

Commit message: update latest production files
Parts:
- J3: Components (none) -> https://www.digikey.com/en/products/detail/sparkfun-electro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
Changed lines of the file:
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@@
       (effects (font (size 0.508 0.508)) hide)
     )
-    (property "Datasheet" "https://www.digikey.com/en/products/detail/amphenol-cs-fci/MDT420E03001/5810340" (id 3) (at 313.69 194.31 0)
+    (property "Datasheet" "https://www.digikey.com/en/products/detail/te-connectivity-amp-connectors/2199230-4/4208915" (id 3) (at 313.69 194.31 0)
       (effects (font (size 1.27 1.27)) hide)
     )
+    (property "Components" "https://www.digikey.com/en/products/detail/sparkfun-electronics/KIT-16549/13282888" (id 4) (at 313.69 194.31 0)
+      (effects (font (size 1.27 1.27)) hide)
+    )

Commit message: add key scan notes to schematic
Other:
- note added: "Basic Key Scan Operation: 1. Set nMATRIX_LD high to enable SIPO write 2. Write to SIPO to set one row low and others high 3. Set nMATRIX_LD low to store column values in PISOs 4. Set nMATRIX_LD high to enable PISO read 5. Read column values from PISO 6. Repeat steps 2-5 for all rows"
- note added: "Key Interrupt Operation: 1. Set all rows low 2. When any key is pressed nKEY_INT will be pulled low and trigger interrupt 3. Disable interrupt, set all rows high, start scan routine"
- note added: "SPI can be used to simplify and speed up shift register reads/writes. Bus cannot currently be shared with other SPI devices because shift register output is not tri-state."
- note removed: "Key interrupt operation: 1. Set all rows low 2. When any key is pressed nKEY_INT will be pulled low and trigger interrupt 3. Disable interrupt, set all rows high, start scan routine..."
- note removed: "Note: nMATRIX_LD should be low for PISO enable and high for SIPO enable"
- note removed: "SPI is used to simplify and speed up shift register reads/writes. Bus cannot currently be shared with other SPI devices because shift register output is not tri-state."
Changed lines of the file:
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@@
     (effects (font (size 2 2) (thickness 0.4) bold) (justify left bottom))
   )
-  (text "Key interrupt operation:\n1. Set all rows low\n2. When any key is pressed nKEY_INT will be pulled low\n   and trigger interrupt\n3. Disable interrupt, set all rows high, start scan routine..."
+  (text "Key Interrupt Operation:\n1. Set all rows low\n2. When any key is pressed nKEY_INT will be pulled low\n   and trigger interrupt\n3. Disable interrupt, set all rows high, start scan routine"
     (at 219.71 281.94 0)
     (effects (font (size 1.27 1.27)) (justify left bottom))
@@
     (effects (font (size 2 2) (thickness 0.4) bold) (justify left bottom))
   )
-  (text "SPI is used to\nsimplify and speed up\nshift register reads/writes.\nBus cannot currently be shared with\nother SPI devices because shift\nregister output is not tri-state."
+  (text "SPI can be used to\nsimplify and speed up\nshift register reads/writes.\nBus cannot currently be shared with\nother SPI devices because shift\nregister output is not tri-state."
     (at 342.9 140.97 0)
     (effects (font (size 1.27 1.27)) (justify left bottom))
@@
     (effects (font (size 2 2) (thickness 0.4) bold) (justify right bottom))
   )
-  (text "Note: nMATRIX_LD should be low for PISO enable and high for SIPO enable"
-    (at 88.9 93.98 0)
+  (text "Basic Key Scan Operation:\n1. Set nMATRIX_LD high to enable SIPO write\n2. Write to SIPO to set one row low and others high\n3. Set nMATRIX_LD low to store column values in PISOs\n4. Set nMATRIX_LD high to enable PISO read\n5. Read column values from PISO\n6. Repeat steps 2-5 for all rows"
+    (at 78.74 41.91 0)
     (effects (font (size 1.27 1.27)) (justify left bottom))
   )
